File: kicad/MAP4.kicad_pcb (KiCad board)
At the start: 2 copper layers, 60 x 34 mm, 9 parts, among them P2 Pin

Commit message: added assembly images
Parts:
- kibuzzard-655707C1: footprint kibuzzard-655707C1 -> map4_fp:kibuzzard-655707C1
Changed lines of the file:
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@@
     (grid_origin 100 100)
     (pcbplotparams
-      (layerselection 0x0000130_ffffffff)
-      (plot_on_all_layers_selection 0x0001000_00000000)
+      (layerselection 0x0000030_7ffffffe)
+      (plot_on_all_layers_selection 0x0000000_00000000)
       (disableapertmacros false)
       (usegerberextensions false)
@@
       (hpglpendiameter 15.000000)
       (dxfpolygonmode true)
-      (dxfimperialunits true)
+      (dxfimperialunits false)
       (dxfusepcbnewfont true)
       (psnegative false)
@@
       (sketchpadsonfab false)
       (subtractmaskfromsilk true)
-      (outputformat 4)
+      (outputformat 3)
       (mirror false)
       (drillshape 2)
@@
     (pad "2" thru_hole circle (at 1.27 0 180) (size 1.8 1.8) (drill 0.8) (layers "*.Cu" "*.Mask" "F.SilkS")
       (net 3 "/LED_red") (pinfunction "K") (pintype "passive"))
-    (model "${KIPRJMOD}/3d_modules/LED_5mm.wrl"
+    (model "${KIPRJMOD}/3d_modules/LED_5mm.step"
       (offset (xyz 0 0 0))
       (scale (xyz 1 1 1))
@@
     (pad "2" thru_hole circle (at 4.064 0 90) (size 1.6 1.6) (drill 0.8) (layers "*.Cu" "*.Mask" "B.SilkS")
       (net 3 "/LED_red") (pintype "passive"))
-    (model "${KIPRJMOD}/3d_modules/resistor_7_62mm.wrl"
+    (model "${KIPRJMOD}/3d_modules/resistor_7_62mm.step"
       (offset (xyz 0 0 0))
       (scale (xyz 1 1 1))
@@
     (pad "2" thru_hole circle (at 0 13 270) (size 2.5 2.5) (drill 1.3) (layers "*.Cu" "*.Mask" "B.SilkS")
       (net 2 "/GND") (pinfunction "-") (pintype "passive"))
-    (model "CR2032_HOR_HOLD.wrl"
-      (offset (xyz 0 0 0))
-      (scale (xyz 1 1 1))
-      (rotate (xyz 0 0 0))
-    )
-  )
-  (footprint "kibuzzard-655707C1" (layer "B.Cu")
+    (model "${KIPRJMOD}/3d_modules/CR2032_HOR_HOLD.step"
+      (offset (xyz 0 0 0))
+      (scale (xyz 1 1 1))
+      (rotate (xyz 0 0 0))
+    )
+  )
+  (footprint "map4_fp:kibuzzard-655707C1" (layer "B.Cu")
     (at 112.4 69 180)
     (descr "Generated with KiBuzzard")
